File: pcbs/fourStages1.sch (KiCad schematic (older format))
At the start: 12 parts, among them Q1 MMBT3904, Q2 MMBT3904, Q3 MMBT3904, Q4 MMBT3904, U1 LM324DT

Commit message: Started layouting.
Parts:
- removed C2: 100n, Resistors_SMD:R_0603, symbol C
- removed Q1, Q2, Q3, Q4: MMBT3904, SOT-23, symbol MMBT3904
- removed R1, R2, R3, R4: 10R, Resistors_SMD:R_0603, symbol R
- removed U1: LM324DT, SMD_Packages:SOIC-14_N, symbol LM324DT
- added C?: 1u, Resistors_SMD:R_0603, symbol C
- added C?: 10n, Resistors_SMD:R_0603, symbol C
- added Q? (x2): MBT3904DW1, TO_SOT_Packages_SMD:SOT-363, symbol MBT3904DW1
- added R? (x2): 10R, Resistors_SMD:R_0603, symbol R
- added R? (x2): 180k, Resistors_SMD:R_0603, symbol R
- added R? (x2): 20k, Resistors_SMD:R_0603, symbol R
- added R? (x2): 10k, Resistors_SMD:R_0603, symbol R
- added U? (x4): LM324QT, QFN:QFN-16-1EP_3x3mm_Pitch0.5mm_ThermalVias, symbol LM324QT
- C1: Digikey (none) -> 445-5146-1-ND; Farnell 2496916 -> (none)
- C3: Digikey (none) -> 490-7194-1-ND; Farnell 1414609 -> (none)
Connections:
- net labels removed: LED_NEG_2, LED_NEG_3, LED_NEG_4
- wire segments 37 -> 42
Other:
- moved on the sheet: C1, C3
