File: pcbs/led_driver.sch (KiCad schematic (older format))
At the start: 5 parts

Commit message: Started layouting.
Parts:
- removed CON?: BARREL_JACK, symbol BARREL_JACK
- removed P? (x2): CONN_01X03, symbol CONN_01X03
- removed R?: 160k, symbol R
- removed R?: 1.8k, symbol R
Connections:
- net labels removed: GND, VSIG, Vcc
- wire segments 10 -> 0
Changed lines of the file:
@@
 LIBS:contrib
 LIBS:valves
-LIBS:myOpAmps
+LIBS:myopamps
 EELAYER 25 0
 EELAYER END
 $Descr A4 11693 8268
 encoding utf-8
-Sheet 1 2
+Sheet 1 18
 Title ""
 Date ""
@@
 $EndDescr
 $Sheet
-S 3600 2375 1200 1125
-U 5946A580
-F0 "fourStages1" 60
-F1 "fourStages1.sch" 60
-F2 "LED_NEG_3" I L 3600 3000 60
-F3 "LED_NEG_1" I L 3600 2600 60
-F4 "LED_NEG_4" I L 3600 3200 60
-F5 "LED_NEG_2" I L 3600 2800 60
+S 6400 1875 2125 2050
+U 5A0916C5
+F0 "LEDDriver" 60
+F1 "LEDDriver.sch" 60
 $EndSheet
-$Comp
-L BARREL_JACK CON?
-U 1 1 59468F94
-P 1900 1400
-F 0 "CON?" H 1900 1650 50  0000 C CNN
-F 1 "BARREL_JACK" H 1900 1200 50  0000 C CNN
-F 2 "" H 1900 1400 50  0000 C CNN
-F 3 "" H 1900 1400 50  0000 C CNN
-	1    1900 1400
-	1    0    0    -1
-$EndComp
-Text GLabel 2725 1300 2    60   Output ~ 0
-Vcc
-Wire Wire Line
-	2200 1300 2725 1300
-$Comp
-L PWR_FLAG #FLG?
-U 1 1 5946963E
-P 2350 1175
-F 0 "#FLG?" H 2350 1270 50  0001 C CNN
-F 1 "PWR_FLAG" H 2350 1355 50  0000 C CNN
-F 2 "" H 2350 1175 50  0000 C CNN
-F 3 "" H 2350 1175 50  0000 C CNN
-	1    2350 1175
-	1    0    0    -1
-$EndComp
-Wire Wire Line
-	2350 1175 2350 1300
-Connection ~ 2350 1300
-$Comp
-L GND #PWR?
-U 1 1 594697AB
-P 2700 1625
-F 0 "#PWR?" H 2700 1375 50  0001 C CNN
-F 1 "GND" H 2700 1475 50  0000 C CNN
-F 2 "" H 2700 1625 50  0000 C CNN
-F 3 "" H 2700 1625 50  0000 C CNN
-	1    2700 1625
-	1    0    0    -1
-$EndComp
-Wire Wire Line
-	2200 1500 2700 1500
-Wire Wire Line
-	2700 1500 2700 1625
-Wire Wire Line
-	2200 1400 2350 1400
-Wire Wire Line
-	2350 1400 2350 1600
-Connection ~ 2350 1500
-$Comp
-L PWR_FLAG #FLG?
-U 1 1 59469875
-P 2350 1600
-F 0 "#FLG?" H 2350 1695 50  0001 C CNN
-F 1 "PWR_FLAG" H 2350 1780 50  0000 C CNN
-F 2 "" H 2350 1600 50  0000 C CNN
-F 3 "" H 2350 1600 50  0000 C CNN
-	1    2350 1600
-	-1   0    0    1
-$EndComp
-$Comp
-L R R?
-U 1 1 5946A551
-P 6425 1150
-F 0 "R?" V 6505 1150 50  0000 C CNN
-F 1 "160k" V 6425 1150 50  0000 C CNN
-F 2 "" V 6355 1150 50  0000 C CNN
-F 3 "" H 6425 1150 50  0000 C CNN
-	1    6425 1150
-	1    0    0    -1
-$EndComp
-$Comp
-L CONN_01X03 P?
-U 1 1 5946AAD6
-P 7900 1250
-F 0 "P?" H 7900 1450 50  0000 C CNN
-F 1 "CONN_01X03" V 8000 1250 50  0000 C CNN
-F 2 "" H 7900 1250 50  0000 C CNN
-F 3 "" H 7900 1250 50  0000 C CNN
-	1    7900 1250
-	1    0    0    -1
-$EndComp
-$Comp
-L R R?
-U 1 1 5946AB9F
-P 6425 1575
-F 0 "R?" V 6505 1575 50  0000 C CNN
-F 1 "1.8k" V 6425 1575 50  0000 C CNN
-F 2 "" V 6355 1575 50  0000 C CNN
-F 3 "" H 6425 1575 50  0000 C CNN
-	1    6425 1575
-	1    0    0    -1
-$EndComp
-$Comp
-L CONN_01X03 P?
-U 1 1 5946AC97
-P 8250 1250
-F 0 "P?" H 8250 1450 50  0000 C CNN
-F 1 "CONN_01X03" V 8350 1250 50  0000 C CNN
-F 2 "" H 8250 1250 50  0000 C CNN
-F 3 "" H 8250 1250 50  0000 C CNN
-	1    8250 1250
-	-1   0    0    -1
-$EndComp
-Text GLabel 8725 1250 2    60   Output ~ 0
-VSIG
-Wire Wire Line
-	8725 1250 8450 1250
-Wire Wire Line
-	8450 1150 8575 1150
-Wire Wire Line
-	8575 1150 8575 1350
-Connection ~ 8575 1250
-Wire Wire Line
-	8575 1350 8450 1350
 $EndSCHEMATC
