File: pcbs/4Stages1.sch (KiCad schematic (older format))
At the start: 14 parts, among them Q1 MBT3904DW1, U1 LM324QT

Commit message: LED driver part done.
Changed lines of the file:
@@
 LIBS:valves
 LIBS:myopamps
+LIBS:led_driver-cache
 EELAYER 25 0
 EELAYER END
 $Descr A4 11693 8268
 encoding utf-8
-Sheet 10 18
+Sheet 3 4
 Title "LED Driver Single Stage"
 Date "2017-11-12"
@@
 AR Path="/5A0916C5/5A0BB0FD/5946B2F2" Ref="C57"  Part="1"
 AR Path="/5A0916C5/5A0BB101/5946B2F2" Ref="C61"  Part="1"
-F 0 "C29" H 5725 1875 50  0000 L CNN
+F 0 "C1" H 5725 1875 50  0000 L CNN
 F 1 "1u" H 5725 1675 50  0000 L CNN
 F 2 "Resistors_SMD:R_0603" H 5738 1625 50  0001 C CNN
@@
 AR Path="/5A0916C5/5A0BB0FD/5946B3BE" Ref="C59"  Part="1"
 AR Path="/5A0916C5/5A0BB101/5946B3BE" Ref="C63"  Part="1"
-F 0 "C31" H 6000 1875 50  0000 L CNN
+F 0 "C3" H 6000 1875 50  0000 L CNN
 F 1 "10n" H 6000 1675 50  0000 L CNN
 F 2 "Resistors_SMD:R_0603" H 6013 1625 50  0001 C CNN
@@
 AR Path="/5A0916C5/5A0BB0FD/5946B480" Ref="#PWR174"  Part="1"
 AR Path="/5A0916C5/5A0BB101/5946B480" Ref="#PWR186"  Part="1"
-F 0 "#PWR90" H 5975 1750 50  0001 C CNN
+F 0 "#PWR6" H 5975 1750 50  0001 C CNN
 F 1 "GND" H 5975 1850 50  0000 C CNN
 F 2 "" H 5975 2000 50  0000 C CNN
@@
 AR Path="/5A0916C5/5A0BB0FD/5A086E54" Ref="Q15"  Part="1"
 AR Path="/5A0916C5/5A0BB101/5A086E54" Ref="Q16"  Part="1"
-F 0 "Q8" H 5350 3500 50  0000 L CNN
+F 0 "Q1" H 5350 3500 50  0000 L CNN
 F 1 "MBT3904DW1" H 5350 3400 50  0000 L CNN
 F 2 "TO_SOT_Packages_SMD:SOT-363_SC-70-6" H 5350 3550 50  0001 C CNN
@@
 AR Path="/5A0916C5/5A0BB0FD/5A087AFB" Ref="R116"  Part="1"
 AR Path="/5A0916C5/5A0BB101/5A087AFB" Ref="R124"  Part="1"
-F 0 "R60" V 5330 4725 50  0000 C CNN
+F 0 "R4" V 5330 4725 50  0000 C CNN
 F 1 "10R" V 5250 4725 50  0000 C CNN
 F 2 "Resistors_SMD:R_0603" V 5180 4725 50  0001 C CNN
@@
 AR Path="/5A0916C5/5A0BB0FD/5A0888D1" Ref="R114"  Part="1"
 AR Path="/5A0916C5/5A0BB101/5A0888D1" Ref="R122"  Part="1"
-F 0 "R58" V 4430 5050 50  0000 C CNN
+F 0 "R2" V 4430 5050 50  0000 C CNN
 F 1 "180k" V 4350 5050 50  0000 C CNN
 F 2 "Resistors_SMD:R_0603" V 4280 5050 50  0001 C CNN
@@
 AR Path="/5A0916C5/5A0BB0FD/5A088CA7" Ref="R115"  Part="1"
 AR Path="/5A0916C5/5A0BB101/5A088CA7" Ref="R123"  Part="1"
-F 0 "R59" V 4930 4575 50  0000 C CNN
+F 0 "R3" V 4930 4575 50  0000 C CNN
 F 1 "20k" V 4850 4575 50  0000 C CNN
 F 2 "Resistors_SMD:R_0603" V 4780 4575 50  0001 C CNN
@@
 AR Path="/5A0916C5/5A0BB0FD/5A088F17" Ref="#PWR169"  Part="1"
 AR Path="/5A0916C5/5A0BB101/5A088F17" Ref="#PWR181"  Part="1"
-F 0 "#PWR85" H 3700 3525 50  0001 C CNN
+F 0 "#PWR1" H 3700 3525 50  0001 C CNN
 F 1 "GND" H 3700 3625 50  0000 C CNN
 F 2 "" H 3700 3775 50  0001 C CNN
@@
 AR Path="/5A0916C5/5A0BB0FD/5A08A1AF" Ref="U15"  Part="2"
 AR Path="/5A0916C5/5A0BB101/5A08A1AF" Ref="U16"  Part="2"
-F 0 "U8" H 4450 3650 50  0000 L CNN
+F 0 "U1" H 4450 3650 50  0000 L CNN
 F 1 "LM324QT" H 4450 3250 50  0000 L CNN
 F 2 "QFN:QFN-16-1EP_3x3mm_Pitch0.5mm_ThermalVias" H 4400 3550 50  0001 C CNN
@@
 AR Path="/5A0916C5/5A0BB0FD/5A08A9A7" Ref="U15"  Part="1"
 AR Path="/5A0916C5/5A0BB101/5A08A9A7" Ref="U16"  Part="1"
-F 0 "U8" H 4250 4675 50  0000 L CNN
+F 0 "U1" H 4250 4675 50  0000 L CNN
 F 1 "LM324QT" H 4250 4275 50  0000 L CNN
 F 2 "QFN:QFN-16-1EP_3x3mm_Pitch0.5mm_ThermalVias" H 4200 4575 50  0001 C CNN
@@
 AR Path="/5A0916C5/5A0BB0FD/5A08B1A6" Ref="#PWR170"  Part="1"
 AR Path="/5A0916C5/5A0BB101/5A08B1A6" Ref="#PWR182"  Part="1"
-F 0 "#PWR86" H 4350 3500 50  0001 C CNN
+F 0 "#PWR2" H 4350 3500 50  0001 C CNN
 F 1 "GND" H 4350 3600 50  0000 C CNN
 F 2 "" H 4350 3750 50  0001 C CNN
@@
 AR Path="/5A0916C5/5A0BB0FD/5A08B22F" Ref="#PWR171"  Part="1"
 AR Path="/5A0916C5/5A0BB101/5A08B22F" Ref="#PWR183"  Part="1"
-F 0 "#PWR87" H 4350 4525 50  0001 C CNN
+F 0 "#PWR3" H 4350 4525 50  0001 C CNN
 F 1 "GND" H 4350 4625 50  0000 C CNN
 F 2 "" H 4350 4775 50  0001 C CNN
@@
 AR Path="/5A0916C5/5A0BB0FD/5A08BC5E" Ref="#PWR172"  Part="1"
 AR Path="/5A0916C5/5A0BB101/5A08BC5E" Ref="#PWR184"  Part="1"
-F 0 "#PWR88" H 5050 4725 50  0001 C CNN
+F 0 "#PWR4" H 5050 4725 50  0001 C CNN
 F 1 "GND" H 5050 4825 50  0000 C CNN
 F 2 "" H 5050 4975 50  0001 C CNN
@@
 AR Path="/5A0916C5/5A0BB0FD/5A08BE2E" Ref="#PWR173"  Part="1"
 AR Path="/5A0916C5/5A0BB101/5A08BE2E" Ref="#PWR185"  Part="1"
-F 0 "#PWR89" H 5250 4725 50  0001 C CNN
+F 0 "#PWR5" H 5250 4725 50  0001 C CNN
 F 1 "GND" H 5250 4825 50  0000 C CNN
 F 2 "" H 5250 4975 50  0001 C CNN
@@
 AR Path="/5A0916C5/5A0BB0FD/5A08C750" Ref="R113"  Part="1"
 AR Path="/5A0916C5/5A0BB101/5A08C750" Ref="R121"  Part="1"
-F 0 "R57" V 3780 3550 50  0000 C CNN
+F 0 "R1" V 3780 3550 50  0000 C CNN
 F 1 "10k" V 3700 3550 50  0000 C CNN
 F 2 "Resistors_SMD:R_0603" V 3630 3550 50  0001 C CNN
@@
 AR Path="/5A0916C5/5A0BB0FD/5A08DFE4" Ref="Q15"  Part="2"
 AR Path="/5A0916C5/5A0BB101/5A08DFE4" Ref="Q16"  Part="2"
-F 0 "Q8" H 6850 3500 50  0000 L CNN
+F 0 "Q1" H 6850 3500 50  0000 L CNN
 F 1 "MBT3904DW1" H 6850 3400 50  0000 L CNN
 F 2 "TO_SOT_Packages_SMD:SOT-363_SC-70-6" H 6850 3550 50  0001 C CNN
@@
 AR Path="/5A0916C5/5A0BB0FD/5A08DFEB" Ref="R117"  Part="1"
 AR Path="/5A0916C5/5A0BB101/5A08DFEB" Ref="R125"  Part="1"
-F 0 "R61" V 6630 4725 50  0000 C CNN
+F 0 "R5" V 6630 4725 50  0000 C CNN
 F 1 "10R" V 6550 4725 50  0000 C CNN
 F 2 "Resistors_SMD:R_0603" V 6480 4725 50  0001 C CNN
@@
 AR Path="/5A0916C5/5A0BB0FD/5A08DFF3" Ref="R119"  Part="1"
 AR Path="/5A0916C5/5A0BB101/5A08DFF3" Ref="R127"  Part="1"
-F 0 "R63" V 7530 5050 50  0000 C CNN
+F 0 "R7" V 7530 5050 50  0000 C CNN
 F 1 "180k" V 7450 5050 50  0000 C CNN
 F 2 "Resistors_SMD:R_0603" V 7380 5050 50  0001 C CNN
@@
 AR Path="/5A0916C5/5A0BB0FD/5A08DFFA" Ref="R118"  Part="1"
 AR Path="/5A0916C5/5A0BB101/5A08DFFA" Ref="R126"  Part="1"
-F 0 "R62" V 7030 4575 50  0000 C CNN
+F 0 "R6" V 7030 4575 50  0000 C CNN
 F 1 "20k" V 6950 4575 50  0000 C CNN
 F 2 "Resistors_SMD:R_0603" V 6880 4575 50  0001 C CNN
@@
 AR Path="/5A0916C5/5A0BB0FD/5A08E000" Ref="#PWR180"  Part="1"
 AR Path="/5A0916C5/5A0BB101/5A08E000" Ref="#PWR192"  Part="1"
-F 0 "#PWR96" H 8100 3525 50  0001 C CNN
+F 0 "#PWR12" H 8100 3525 50  0001 C CNN
 F 1 "GND" H 8100 3625 50  0000 C CNN
 F 2 "" H 8100 3775 50  0001 C CNN
@@
 AR Path="/5A0916C5/5A0BB0FD/5A08E007" Ref="U15"  Part="3"
 AR Path="/5A0916C5/5A0BB101/5A08E007" Ref="U16"  Part="3"
-F 0 "U8" H 7350 3650 50  0000 L CNN
+F 0 "U1" H 7350 3650 50  0000 L CNN
 F 1 "LM324QT" H 7350 3250 50  0000 L CNN
 F 2 "QFN:QFN-16-1EP_3x3mm_Pitch0.5mm_ThermalVias" H 7300 3550 50  0001 C CNN
@@
 AR Path="/5A0916C5/5A0BB0FD/5A08E00E" Ref="U15"  Part="4"
 AR Path="/5A0916C5/5A0BB101/5A08E00E" Ref="U16"  Part="4"
-F 0 "U8" H 7550 4675 50  0000 L CNN
+F 0 "U1" H 7550 4675 50  0000 L CNN
 F 1 "LM324QT" H 7550 4275 50  0000 L CNN
 F 2 "QFN:QFN-16-1EP_3x3mm_Pitch0.5mm_ThermalVias" H 7500 4575 50  0001 C CNN
@@
 AR Path="/5A0916C5/5A0BB0FD/5A08E015" Ref="#PWR178"  Part="1"
 AR Path="/5A0916C5/5A0BB101/5A08E015" Ref="#PWR190"  Part="1"
-F 0 "#PWR94" H 7450 3500 50  0001 C CNN
+F 0 "#PWR10" H 7450 3500 50  0001 C CNN
 F 1 "GND" H 7450 3600 50  0000 C CNN
 F 2 "" H 7450 3750 50  0001 C CNN
@@
 AR Path="/5A0916C5/5A0BB0FD/5A08E01B" Ref="#PWR179"  Part="1"
 AR Path="/5A0916C5/5A0BB101/5A08E01B" Ref="#PWR191"  Part="1"
-F 0 "#PWR95" H 7450 4525 50  0001 C CNN
+F 0 "#PWR11" H 7450 4525 50  0001 C CNN
 F 1 "GND" H 7450 4625 50  0000 C CNN
 F 2 "" H 7450 4775 50  0001 C CNN
@@
 AR Path="/5A0916C5/5A0BB0FD/5A08E02C" Ref="#PWR177"  Part="1"
 AR Path="/5A0916C5/5A0BB101/5A08E02C" Ref="#PWR189"  Part="1"
-F 0 "#PWR93" H 6750 4725 50  0001 C CNN
+F 0 "#PWR9" H 6750 4725 50  0001 C CNN
 F 1 "GND" H 6750 4825 50  0000 C CNN
 F 2 "" H 6750 4975 50  0001 C CNN
@@
 AR Path="/5A0916C5/5A0BB0FD/5A08E038" Ref="#PWR176"  Part="1"
 AR Path="/5A0916C5/5A0BB101/5A08E038" Ref="#PWR188"  Part="1"
-F 0 "#PWR92" H 6550 4725 50  0001 C CNN
+F 0 "#PWR8" H 6550 4725 50  0001 C CNN
 F 1 "GND" H 6550 4825 50  0000 C CNN
 F 2 "" H 6550 4975 50  0001 C CNN
@@
 AR Path="/5A0916C5/5A0BB0FD/5A08E043" Ref="R120"  Part="1"
 AR Path="/5A0916C5/5A0BB101/5A08E043" Ref="R128"  Part="1"
-F 0 "R64" V 8180 3550 50  0000 C CNN
+F 0 "R8" V 8180 3550 50  0000 C CNN
 F 1 "10k" V 8100 3550 50  0000 C CNN
 F 2 "Resistors_SMD:R_0603" V 8030 3550 50  0001 C CNN
@@
 AR Path="/5A0916C5/5A0BB0FD/5A08FEA2" Ref="C58"  Part="1"
 AR Path="/5A0916C5/5A0BB101/5A08FEA2" Ref="C62"  Part="1"
-F 0 "C30" H 5750 2550 50  0000 L CNN
+F 0 "C2" H 5750 2550 50  0000 L CNN
 F 1 "1u" H 5750 2350 50  0000 L CNN
 F 2 "Resistors_SMD:R_0603" H 5763 2300 50  0001 C CNN
@@
 AR Path="/5A0916C5/5A0BB0FD/5A08FEA9" Ref="C60"  Part="1"
 AR Path="/5A0916C5/5A0BB101/5A08FEA9" Ref="C64"  Part="1"
-F 0 "C32" H 6025 2550 50  0000 L CNN
+F 0 "C4" H 6025 2550 50  0000 L CNN
 F 1 "10n" H 6025 2350 50  0000 L CNN
 F 2 "Resistors_SMD:R_0603" H 6038 2300 50  0001 C CNN
@@
 AR Path="/5A0916C5/5A0BB0FD/5A08FEAF" Ref="#PWR175"  Part="1"
 AR Path="/5A0916C5/5A0BB101/5A08FEAF" Ref="#PWR187"  Part="1"
-F 0 "#PWR91" H 6000 2425 50  0001 C CNN
+F 0 "#PWR7" H 6000 2425 50  0001 C CNN
 F 1 "GND" H 6000 2525 50  0000 C CNN
 F 2 "" H 6000 2675 50  0000 C CNN
