File: pcbs/proj/UI.sch (KiCad schematic (older format))
At the start: 21 parts, among them J8 Conn_01x07, SW1 MY_SW_Push_Dual, SW2 Rotary_Encoder, SW3 Rotary_Encoder

Commit message: All components placed.
Parts:
- SW2, SW3: footprint MyTactileSW:ROT_ENC_EN12_TT_Electronics_No_Switch -> MySWs:ROT_ENC_EN12_TT_Electronics_No_Switch
Changed lines of the file:
@@
 Connection ~ 3125 4550
 $Comp
-L GND #PWR0332
+L GND #PWR0300
 U 1 1 5A0B85D7
 P 3875 4575
-F 0 "#PWR0332" H 3875 4325 50  0001 C CNN
+F 0 "#PWR0300" H 3875 4325 50  0001 C CNN
 F 1 "GND" H 3875 4425 50  0000 C CNN
 F 2 "" H 3875 4575 50  0001 C CNN
@@
 Connection ~ 2950 4550
 $Comp
-L Rotary_Encoder SW3
-U 1 1 5A0B8D30
-P 7900 4825
-F 0 "SW3" H 7900 5085 50  0000 C CNN
-F 1 "Rotary_Encoder" H 7900 4565 50  0000 C CNN
-F 2 "MyTactileSW:ROT_ENC_EN12_TT_Electronics_No_Switch" H 7800 4985 50  0001 C CNN
-F 3 "http://www.ttelectronics.com/sites/default/files/download-files/Datasheet_RotaryEncoder_EN12Series.pdf" H 7900 5085 50  0001 C CNN
-F 4 "987-1399-ND" H 7900 4825 60  0001 C CNN "Digikey"
-	1    7900 4825
-	0    1    1    0
-$EndComp
-$Comp
-L GND #PWR0333
+L GND #PWR0301
 U 1 1 5A0B9013
 P 8075 4125
-F 0 "#PWR0333" H 8075 3875 50  0001 C CNN
+F 0 "#PWR0301" H 8075 3875 50  0001 C CNN
 F 1 "GND" H 8075 3975 50  0000 C CNN
 F 2 "" H 8075 4125 50  0001 C CNN
@@
 $EndComp
 $Comp
-L GND #PWR0334
+L GND #PWR0302
 U 1 1 5A0BA939
 P 8825 4850
-F 0 "#PWR0334" H 8825 4600 50  0001 C CNN
+F 0 "#PWR0302" H 8825 4600 50  0001 C CNN
 F 1 "GND" H 8825 4700 50  0000 C CNN
 F 2 "" H 8825 4850 50  0001 C CNN
@@
 $EndComp
 $Comp
-L GND #PWR0335
+L GND #PWR0303
 U 1 1 5A0BE4A9
 P 6975 4850
-F 0 "#PWR0335" H 6975 4600 50  0001 C CNN
+F 0 "#PWR0303" H 6975 4600 50  0001 C CNN
 F 1 "GND" H 6975 4700 50  0000 C CNN
 F 2 "" H 6975 4850 50  0001 C CNN
@@
 F 0 "SW2" H 7845 3515 50  0000 C CNN
 F 1 "Rotary_Encoder" H 7845 2995 50  0000 C CNN
-F 2 "MyTactileSW:ROT_ENC_EN12_TT_Electronics_No_Switch" H 7745 3415 50  0001 C CNN
+F 2 "MySWs:ROT_ENC_EN12_TT_Electronics_No_Switch" H 7745 3415 50  0001 C CNN
 F 3 "http://www.ttelectronics.com/sites/default/files/download-files/Datasheet_RotaryEncoder_EN12Series.pdf" H 7845 3515 50  0001 C CNN
 F 4 "987-1399-ND" H 7845 3255 60  0001 C CNN "Digikey"
@@
 $EndComp
 $Comp
-L GND #PWR0336
+L GND #PWR0304
 U 1 1 5A0E5835
 P 8020 2555
-F 0 "#PWR0336" H 8020 2305 50  0001 C CNN
+F 0 "#PWR0304" H 8020 2305 50  0001 C CNN
 F 1 "GND" H 8020 2405 50  0000 C CNN
 F 2 "" H 8020 2555 50  0001 C CNN
@@
 $EndComp
 $Comp
-L GND #PWR0337
+L GND #PWR0305
 U 1 1 5A0E584B
 P 8770 3280
-F 0 "#PWR0337" H 8770 3030 50  0001 C CNN
+F 0 "#PWR0305" H 8770 3030 50  0001 C CNN
 F 1 "GND" H 8770 3130 50  0000 C CNN
 F 2 "" H 8770 3280 50  0001 C CNN
@@
 $EndComp
 $Comp
-L GND #PWR0338
+L GND #PWR0306
 U 1 1 5A0E5872
 P 6920 3280
-F 0 "#PWR0338" H 6920 3030 50  0001 C CNN
+F 0 "#PWR0306" H 6920 3030 50  0001 C CNN
 F 1 "GND" H 6920 3130 50  0000 C CNN
 F 2 "" H 6920 3280 50  0001 C CNN
@@
 $Comp
 L MY_SW_Push_Dual SW1
-U 1 1 5A0DB5F5
+U 1 1 5A0EBF07
 P 3425 4450
 F 0 "SW1" H 3475 4550 50  0000 L CNN
@@
 	1    0    0    -1
 $EndComp
+$Comp
+L Rotary_Encoder SW3
+U 1 1 5A0B8D30
+P 7900 4825
+F 0 "SW3" H 7900 5085 50  0000 C CNN
+F 1 "Rotary_Encoder" H 7900 4565 50  0000 C CNN
+F 2 "MySWs:ROT_ENC_EN12_TT_Electronics_No_Switch" H 7800 4985 50  0001 C CNN
+F 3 "http://www.ttelectronics.com/sites/default/files/download-files/Datasheet_RotaryEncoder_EN12Series.pdf" H 7900 5085 50  0001 C CNN
+F 4 "987-1399-ND" H 7900 4825 60  0001 C CNN "Digikey"
+	1    7900 4825
+	0    1    1    0
+$EndComp
 $EndSCHEMATC
