File: pcbs/proj/2Stages1.sch (KiCad schematic (older format))
At the start: 9 parts, among them Q1 MBT3904DW1, U1 LM324QT

Commit message: Some progress layouting the beast today.
Changed lines of the file:
@@
 $Descr A4 11693 8268
 encoding utf-8
-Sheet 3 37
+Sheet 8 37
 Title "UV LED Driver Two Stages"
 Date "2017-11-13"
@@
 AR Path="/5A0916C5/5A09BEE8/5946B2F2" Ref="C124"  Part="1"
 AR Path="/5A0916C5/5A09BEEC/5946B2F2" Ref="C128"  Part="1"
-F 0 "C20" H 5505 2065 50  0000 L CNN
+F 0 "C24" H 5505 2065 50  0000 L CNN
 F 1 "1u" H 5505 1865 50  0000 L CNN
 F 2 "Resistors_SMD:R_0603" H 5518 1815 50  0001 C CNN
@@
 AR Path="/5A0916C5/5A09BEE8/5A08DFE4" Ref="Q18"  Part="2"
 AR Path="/5A0916C5/5A09BEEC/5A08DFE4" Ref="Q17"  Part="2"
-F 0 "Q5" H 6850 3500 50  0000 L CNN
+F 0 "Q6" H 6850 3500 50  0000 L CNN
 F 1 "MBT3904DW1" H 6850 3400 50  0000 L CNN
 F 2 "TO_SOT_Packages_SMD:SOT-363_SC-70-6" H 6850 3550 50  0001 C CNN
@@
 AR Path="/5A0916C5/5A09BEE8/5A08DFEB" Ref="R188"  Part="1"
 AR Path="/5A0916C5/5A09BEEC/5A08DFEB" Ref="R194"  Part="1"
-F 0 "R32" V 6630 4725 50  0000 C CNN
+F 0 "R38" V 6630 4725 50  0000 C CNN
 F 1 "10R" V 6550 4725 50  0000 C CNN
 F 2 "Resistors_SMD:R_0603" V 6480 4725 50  0001 C CNN
@@
 AR Path="/5A0916C5/5A09BEE8/5A08DFF3" Ref="R190"  Part="1"
 AR Path="/5A0916C5/5A09BEEC/5A08DFF3" Ref="R196"  Part="1"
-F 0 "R34" V 7530 5050 50  0000 C CNN
+F 0 "R40" V 7530 5050 50  0000 C CNN
 F 1 "180k" V 7450 5050 50  0000 C CNN
 F 2 "Resistors_SMD:R_0603" V 7380 5050 50  0001 C CNN
@@
 AR Path="/5A0916C5/5A09BEE8/5A08DFFA" Ref="R189"  Part="1"
 AR Path="/5A0916C5/5A09BEEC/5A08DFFA" Ref="R195"  Part="1"
-F 0 "R33" V 7030 4575 50  0000 C CNN
+F 0 "R39" V 7030 4575 50  0000 C CNN
 F 1 "20k" V 6950 4575 50  0000 C CNN
 F 2 "Resistors_SMD:R_0603" V 6880 4575 50  0001 C CNN
@@
 AR Path="/5A0916C5/5A09BEE8/5A08E007" Ref="U18"  Part="3"
 AR Path="/5A0916C5/5A09BEEC/5A08E007" Ref="U17"  Part="3"
-F 0 "U5" H 7350 3650 50  0000 L CNN
+F 0 "U6" H 7350 3650 50  0000 L CNN
 F 1 "LM324QT" H 7350 3250 50  0000 L CNN
 F 2 "QFN:QFN-16-1EP_3x3mm_Pitch0.5mm" H 7300 3550 50  0001 C CNN
@@
 AR Path="/5A0916C5/5A09BEE8/5A08E00E" Ref="U18"  Part="4"
 AR Path="/5A0916C5/5A09BEEC/5A08E00E" Ref="U17"  Part="4"
-F 0 "U5" H 7550 4675 50  0000 L CNN
+F 0 "U6" H 7550 4675 50  0000 L CNN
 F 1 "LM324QT" H 7550 4275 50  0000 L CNN
 F 2 "QFN:QFN-16-1EP_3x3mm_Pitch0.5mm" H 7500 4575 50  0001 C CNN
@@
 AR Path="/5A0916C5/5A09BEE8/5A08E015" Ref="#PWR0274"  Part="1"
 AR Path="/5A0916C5/5A09BEEC/5A08E015" Ref="#PWR0283"  Part="1"
-F 0 "#PWR040" H 7450 3500 50  0001 C CNN
+F 0 "#PWR049" H 7450 3500 50  0001 C CNN
 F 1 "GND" H 7450 3600 50  0000 C CNN
 F 2 "" H 7450 3750 50  0001 C CNN
@@
 AR Path="/5A0916C5/5A09BEE8/5A08E01B" Ref="#PWR0275"  Part="1"
 AR Path="/5A0916C5/5A09BEEC/5A08E01B" Ref="#PWR0284"  Part="1"
-F 0 "#PWR041" H 7450 4525 50  0001 C CNN
+F 0 "#PWR050" H 7450 4525 50  0001 C CNN
 F 1 "GND" H 7450 4625 50  0000 C CNN
 F 2 "" H 7450 4775 50  0001 C CNN
@@
 AR Path="/5A0916C5/5A09BEE8/5A08E02C" Ref="#PWR0276"  Part="1"
 AR Path="/5A0916C5/5A09BEEC/5A08E02C" Ref="#PWR0285"  Part="1"
-F 0 "#PWR042" H 6750 4725 50  0001 C CNN
+F 0 "#PWR051" H 6750 4725 50  0001 C CNN
 F 1 "GND" H 6750 4825 50  0000 C CNN
 F 2 "" H 6750 4975 50  0001 C CNN
@@
 AR Path="/5A0916C5/5A09BEE8/5A08E038" Ref="#PWR0277"  Part="1"
 AR Path="/5A0916C5/5A09BEEC/5A08E038" Ref="#PWR0286"  Part="1"
-F 0 "#PWR043" H 6550 4725 50  0001 C CNN
+F 0 "#PWR052" H 6550 4725 50  0001 C CNN
 F 1 "GND" H 6550 4825 50  0000 C CNN
 F 2 "" H 6550 4975 50  0001 C CNN
@@
 AR Path="/5A0916C5/5A09BEE8/5A159798" Ref="Q18"  Part="1"
 AR Path="/5A0916C5/5A09BEEC/5A159798" Ref="Q17"  Part="1"
-F 0 "Q5" H 5350 3500 50  0000 L CNN
+F 0 "Q6" H 5350 3500 50  0000 L CNN
 F 1 "MBT3904DW1" H 5350 3400 50  0000 L CNN
 F 2 "TO_SOT_Packages_SMD:SOT-363_SC-70-6" H 5350 3550 50  0001 C CNN
@@
 AR Path="/5A0916C5/5A09BEE8/5A15979F" Ref="R187"  Part="1"
 AR Path="/5A0916C5/5A09BEEC/5A15979F" Ref="R193"  Part="1"
-F 0 "R31" V 5330 4725 50  0000 C CNN
+F 0 "R37" V 5330 4725 50  0000 C CNN
 F 1 "10R" V 5250 4725 50  0000 C CNN
 F 2 "Resistors_SMD:R_0603" V 5180 4725 50  0001 C CNN
@@
 AR Path="/5A0916C5/5A09BEE8/5A1597A7" Ref="R185"  Part="1"
 AR Path="/5A0916C5/5A09BEEC/5A1597A7" Ref="R191"  Part="1"
-F 0 "R29" V 4430 5050 50  0000 C CNN
+F 0 "R35" V 4430 5050 50  0000 C CNN
 F 1 "180k" V 4350 5050 50  0000 C CNN
 F 2 "Resistors_SMD:R_0603" V 4280 5050 50  0001 C CNN
@@
 AR Path="/5A0916C5/5A09BEE8/5A1597AE" Ref="R186"  Part="1"
 AR Path="/5A0916C5/5A09BEEC/5A1597AE" Ref="R192"  Part="1"
-F 0 "R30" V 4930 4575 50  0000 C CNN
+F 0 "R36" V 4930 4575 50  0000 C CNN
 F 1 "20k" V 4850 4575 50  0000 C CNN
 F 2 "Resistors_SMD:R_0603" V 4780 4575 50  0001 C CNN
@@
 AR Path="/5A0916C5/5A09BEE8/5A1597B5" Ref="U18"  Part="2"
 AR Path="/5A0916C5/5A09BEEC/5A1597B5" Ref="U17"  Part="2"
-F 0 "U5" H 4450 3650 50  0000 L CNN
+F 0 "U6" H 4450 3650 50  0000 L CNN
 F 1 "LM324QT" H 4450 3250 50  0000 L CNN
 F 2 "QFN:QFN-16-1EP_3x3mm_Pitch0.5mm" H 4400 3550 50  0001 C CNN
@@
 AR Path="/5A0916C5/5A09BEE8/5A1597BC" Ref="U18"  Part="1"
 AR Path="/5A0916C5/5A09BEEC/5A1597BC" Ref="U17"  Part="1"
-F 0 "U5" H 4250 4675 50  0000 L CNN
+F 0 "U6" H 4250 4675 50  0000 L CNN
 F 1 "LM324QT" H 4250 4275 50  0000 L CNN
 F 2 "QFN:QFN-16-1EP_3x3mm_Pitch0.5mm" H 4200 4575 50  0001 C CNN
@@
 AR Path="/5A0916C5/5A09BEE8/5A1597C3" Ref="#PWR0278"  Part="1"
 AR Path="/5A0916C5/5A09BEEC/5A1597C3" Ref="#PWR0287"  Part="1"
-F 0 "#PWR044" H 4350 3500 50  0001 C CNN
+F 0 "#PWR053" H 4350 3500 50  0001 C CNN
 F 1 "GND" H 4350 3600 50  0000 C CNN
 F 2 "" H 4350 3750 50  0001 C CNN
@@
 AR Path="/5A0916C5/5A09BEE8/5A1597C9" Ref="#PWR0279"  Part="1"
 AR Path="/5A0916C5/5A09BEEC/5A1597C9" Ref="#PWR0288"  Part="1"
-F 0 "#PWR045" H 4350 4525 50  0001 C CNN
+F 0 "#PWR054" H 4350 4525 50  0001 C CNN
 F 1 "GND" H 4350 4625 50  0000 C CNN
 F 2 "" H 4350 4775 50  0001 C CNN
@@
 AR Path="/5A0916C5/5A09BEE8/5A1597DA" Ref="#PWR0280"  Part="1"
 AR Path="/5A0916C5/5A09BEEC/5A1597DA" Ref="#PWR0289"  Part="1"
-F 0 "#PWR046" H 5050 4725 50  0001 C CNN
+F 0 "#PWR055" H 5050 4725 50  0001 C CNN
 F 1 "GND" H 5050 4825 50  0000 C CNN
 F 2 "" H 5050 4975 50  0001 C CNN
@@
 AR Path="/5A0916C5/5A09BEE8/5A1597E6" Ref="#PWR0281"  Part="1"
 AR Path="/5A0916C5/5A09BEEC/5A1597E6" Ref="#PWR0290"  Part="1"
-F 0 "#PWR047" H 5250 4725 50  0001 C CNN
+F 0 "#PWR056" H 5250 4725 50  0001 C CNN
 F 1 "GND" H 5250 4825 50  0000 C CNN
 F 2 "" H 5250 4975 50  0001 C CNN
@@
 AR Path="/5A0916C5/5A09BEE8/5946B480" Ref="#PWR0282"  Part="1"
 AR Path="/5A0916C5/5A09BEEC/5946B480" Ref="#PWR0291"  Part="1"
-F 0 "#PWR048" H 5480 1865 50  0001 C CNN
+F 0 "#PWR057" H 5480 1865 50  0001 C CNN
 F 1 "GND" H 5480 1965 50  0000 C CNN
 F 2 "" H 5480 2115 50  0000 C CNN

Commit message: Started eliminating DRC errors.
Changed lines of the file:
@@
 $Descr A4 11693 8268
 encoding utf-8
-Sheet 8 37
+Sheet 3 37
 Title "UV LED Driver Two Stages"
 Date "2017-11-13"
@@
 AR Path="/5A0916C5/5A09BEE8/5946B2F2" Ref="C124"  Part="1"
 AR Path="/5A0916C5/5A09BEEC/5946B2F2" Ref="C128"  Part="1"
-F 0 "C24" H 5505 2065 50  0000 L CNN
+F 0 "C4" H 5505 2065 50  0000 L CNN
 F 1 "1u" H 5505 1865 50  0000 L CNN
 F 2 "Resistors_SMD:R_0603" H 5518 1815 50  0001 C CNN
@@
 AR Path="/5A0916C5/5A09BEE8/5A08DFE4" Ref="Q18"  Part="2"
 AR Path="/5A0916C5/5A09BEEC/5A08DFE4" Ref="Q17"  Part="2"
-F 0 "Q6" H 6850 3500 50  0000 L CNN
+F 0 "Q1" H 6850 3500 50  0000 L CNN
 F 1 "MBT3904DW1" H 6850 3400 50  0000 L CNN
 F 2 "TO_SOT_Packages_SMD:SOT-363_SC-70-6" H 6850 3550 50  0001 C CNN
@@
 AR Path="/5A0916C5/5A09BEE8/5A08DFEB" Ref="R188"  Part="1"
 AR Path="/5A0916C5/5A09BEEC/5A08DFEB" Ref="R194"  Part="1"
-F 0 "R38" V 6630 4725 50  0000 C CNN
+F 0 "R8" V 6630 4725 50  0000 C CNN
 F 1 "10R" V 6550 4725 50  0000 C CNN
 F 2 "Resistors_SMD:R_0603" V 6480 4725 50  0001 C CNN
@@
 AR Path="/5A0916C5/5A09BEE8/5A08DFF3" Ref="R190"  Part="1"
 AR Path="/5A0916C5/5A09BEEC/5A08DFF3" Ref="R196"  Part="1"
-F 0 "R40" V 7530 5050 50  0000 C CNN
+F 0 "R10" V 7530 5050 50  0000 C CNN
 F 1 "180k" V 7450 5050 50  0000 C CNN
 F 2 "Resistors_SMD:R_0603" V 7380 5050 50  0001 C CNN
@@
 AR Path="/5A0916C5/5A09BEE8/5A08DFFA" Ref="R189"  Part="1"
 AR Path="/5A0916C5/5A09BEEC/5A08DFFA" Ref="R195"  Part="1"
-F 0 "R39" V 7030 4575 50  0000 C CNN
+F 0 "R9" V 7030 4575 50  0000 C CNN
 F 1 "20k" V 6950 4575 50  0000 C CNN
 F 2 "Resistors_SMD:R_0603" V 6880 4575 50  0001 C CNN
@@
 AR Path="/5A0916C5/5A09BEE8/5A08E007" Ref="U18"  Part="3"
 AR Path="/5A0916C5/5A09BEEC/5A08E007" Ref="U17"  Part="3"
-F 0 "U6" H 7350 3650 50  0000 L CNN
+F 0 "U1" H 7350 3650 50  0000 L CNN
 F 1 "LM324QT" H 7350 3250 50  0000 L CNN
 F 2 "QFN:QFN-16-1EP_3x3mm_Pitch0.5mm" H 7300 3550 50  0001 C CNN
@@
 AR Path="/5A0916C5/5A09BEE8/5A08E00E" Ref="U18"  Part="4"
 AR Path="/5A0916C5/5A09BEEC/5A08E00E" Ref="U17"  Part="4"
-F 0 "U6" H 7550 4675 50  0000 L CNN
+F 0 "U1" H 7550 4675 50  0000 L CNN
 F 1 "LM324QT" H 7550 4275 50  0000 L CNN
 F 2 "QFN:QFN-16-1EP_3x3mm_Pitch0.5mm" H 7500 4575 50  0001 C CNN
@@
 AR Path="/5A0916C5/5A09BEE8/5A08E015" Ref="#PWR0274"  Part="1"
 AR Path="/5A0916C5/5A09BEEC/5A08E015" Ref="#PWR0283"  Part="1"
-F 0 "#PWR049" H 7450 3500 50  0001 C CNN
+F 0 "#PWR0283" H 7450 3500 50  0001 C CNN
 F 1 "GND" H 7450 3600 50  0000 C CNN
 F 2 "" H 7450 3750 50  0001 C CNN
@@
 AR Path="/5A0916C5/5A09BEE8/5A08E01B" Ref="#PWR0275"  Part="1"
 AR Path="/5A0916C5/5A09BEEC/5A08E01B" Ref="#PWR0284"  Part="1"
-F 0 "#PWR050" H 7450 4525 50  0001 C CNN
+F 0 "#PWR0284" H 7450 4525 50  0001 C CNN
 F 1 "GND" H 7450 4625 50  0000 C CNN
 F 2 "" H 7450 4775 50  0001 C CNN
@@
 AR Path="/5A0916C5/5A09BEE8/5A08E02C" Ref="#PWR0276"  Part="1"
 AR Path="/5A0916C5/5A09BEEC/5A08E02C" Ref="#PWR0285"  Part="1"
-F 0 "#PWR051" H 6750 4725 50  0001 C CNN
+F 0 "#PWR0285" H 6750 4725 50  0001 C CNN
 F 1 "GND" H 6750 4825 50  0000 C CNN
 F 2 "" H 6750 4975 50  0001 C CNN
@@
 AR Path="/5A0916C5/5A09BEE8/5A08E038" Ref="#PWR0277"  Part="1"
 AR Path="/5A0916C5/5A09BEEC/5A08E038" Ref="#PWR0286"  Part="1"
-F 0 "#PWR052" H 6550 4725 50  0001 C CNN
+F 0 "#PWR0286" H 6550 4725 50  0001 C CNN
 F 1 "GND" H 6550 4825 50  0000 C CNN
 F 2 "" H 6550 4975 50  0001 C CNN
@@
 AR Path="/5A0916C5/5A09BEE8/5A159798" Ref="Q18"  Part="1"
 AR Path="/5A0916C5/5A09BEEC/5A159798" Ref="Q17"  Part="1"
-F 0 "Q6" H 5350 3500 50  0000 L CNN
+F 0 "Q1" H 5350 3500 50  0000 L CNN
 F 1 "MBT3904DW1" H 5350 3400 50  0000 L CNN
 F 2 "TO_SOT_Packages_SMD:SOT-363_SC-70-6" H 5350 3550 50  0001 C CNN
@@
 AR Path="/5A0916C5/5A09BEE8/5A15979F" Ref="R187"  Part="1"
 AR Path="/5A0916C5/5A09BEEC/5A15979F" Ref="R193"  Part="1"
-F 0 "R37" V 5330 4725 50  0000 C CNN
+F 0 "R7" V 5330 4725 50  0000 C CNN
 F 1 "10R" V 5250 4725 50  0000 C CNN
 F 2 "Resistors_SMD:R_0603" V 5180 4725 50  0001 C CNN
@@
 AR Path="/5A0916C5/5A09BEE8/5A1597A7" Ref="R185"  Part="1"
 AR Path="/5A0916C5/5A09BEEC/5A1597A7" Ref="R191"  Part="1"
-F 0 "R35" V 4430 5050 50  0000 C CNN
+F 0 "R5" V 4430 5050 50  0000 C CNN
 F 1 "180k" V 4350 5050 50  0000 C CNN
 F 2 "Resistors_SMD:R_0603" V 4280 5050 50  0001 C CNN
@@
 AR Path="/5A0916C5/5A09BEE8/5A1597AE" Ref="R186"  Part="1"
 AR Path="/5A0916C5/5A09BEEC/5A1597AE" Ref="R192"  Part="1"
-F 0 "R36" V 4930 4575 50  0000 C CNN
+F 0 "R6" V 4930 4575 50  0000 C CNN
 F 1 "20k" V 4850 4575 50  0000 C CNN
 F 2 "Resistors_SMD:R_0603" V 4780 4575 50  0001 C CNN
@@
 AR Path="/5A0916C5/5A09BEE8/5A1597B5" Ref="U18"  Part="2"
 AR Path="/5A0916C5/5A09BEEC/5A1597B5" Ref="U17"  Part="2"
-F 0 "U6" H 4450 3650 50  0000 L CNN
+F 0 "U1" H 4450 3650 50  0000 L CNN
 F 1 "LM324QT" H 4450 3250 50  0000 L CNN
 F 2 "QFN:QFN-16-1EP_3x3mm_Pitch0.5mm" H 4400 3550 50  0001 C CNN
@@
 AR Path="/5A0916C5/5A09BEE8/5A1597BC" Ref="U18"  Part="1"
 AR Path="/5A0916C5/5A09BEEC/5A1597BC" Ref="U17"  Part="1"
-F 0 "U6" H 4250 4675 50  0000 L CNN
+F 0 "U1" H 4250 4675 50  0000 L CNN
 F 1 "LM324QT" H 4250 4275 50  0000 L CNN
 F 2 "QFN:QFN-16-1EP_3x3mm_Pitch0.5mm" H 4200 4575 50  0001 C CNN
@@
 AR Path="/5A0916C5/5A09BEE8/5A1597C3" Ref="#PWR0278"  Part="1"
 AR Path="/5A0916C5/5A09BEEC/5A1597C3" Ref="#PWR0287"  Part="1"
-F 0 "#PWR053" H 4350 3500 50  0001 C CNN
+F 0 "#PWR0287" H 4350 3500 50  0001 C CNN
 F 1 "GND" H 4350 3600 50  0000 C CNN
 F 2 "" H 4350 3750 50  0001 C CNN
@@
 AR Path="/5A0916C5/5A09BEE8/5A1597C9" Ref="#PWR0279"  Part="1"
 AR Path="/5A0916C5/5A09BEEC/5A1597C9" Ref="#PWR0288"  Part="1"
-F 0 "#PWR054" H 4350 4525 50  0001 C CNN
+F 0 "#PWR0288" H 4350 4525 50  0001 C CNN
 F 1 "GND" H 4350 4625 50  0000 C CNN
 F 2 "" H 4350 4775 50  0001 C CNN
@@
 AR Path="/5A0916C5/5A09BEE8/5A1597DA" Ref="#PWR0280"  Part="1"
 AR Path="/5A0916C5/5A09BEEC/5A1597DA" Ref="#PWR0289"  Part="1"
-F 0 "#PWR055" H 5050 4725 50  0001 C CNN
+F 0 "#PWR0289" H 5050 4725 50  0001 C CNN
 F 1 "GND" H 5050 4825 50  0000 C CNN
 F 2 "" H 5050 4975 50  0001 C CNN
@@
 AR Path="/5A0916C5/5A09BEE8/5A1597E6" Ref="#PWR0281"  Part="1"
 AR Path="/5A0916C5/5A09BEEC/5A1597E6" Ref="#PWR0290"  Part="1"
-F 0 "#PWR056" H 5250 4725 50  0001 C CNN
+F 0 "#PWR0290" H 5250 4725 50  0001 C CNN
 F 1 "GND" H 5250 4825 50  0000 C CNN
 F 2 "" H 5250 4975 50  0001 C CNN
@@
 AR Path="/5A0916C5/5A09BEE8/5946B480" Ref="#PWR0282"  Part="1"
 AR Path="/5A0916C5/5A09BEEC/5946B480" Ref="#PWR0291"  Part="1"
-F 0 "#PWR057" H 5480 1865 50  0001 C CNN
+F 0 "#PWR0291" H 5480 1865 50  0001 C CNN
 F 1 "GND" H 5480 1965 50  0000 C CNN
 F 2 "" H 5480 2115 50  0000 C CNN
