File: pcbs/proj/InterfaceNucleoF103RB.sch (KiCad schematic (older format))
At the start: 8 parts, among them J6 Conn_02x19_Odd_Even, J7 Conn_02x19_Odd_Even

Commit message: Started eliminating DRC errors.
Connections:
- net LIGHT_INT: now reaches J6.3 (Pin_3)
- no-connect marks 56 -> 55
Changed lines of the file:
@@
 NoConn ~ 3130 2965
 NoConn ~ 3130 2865
-NoConn ~ 2630 2765
 NoConn ~ 2630 3165
 NoConn ~ 2630 3265
@@
 NoConn ~ 2630 3465
 NoConn ~ 3130 3965
+Text GLabel 2630 2765 0    47   UnSpc ~ 0
+PD2
+Text GLabel 2405 6590 0    47   UnSpc ~ 0
+PD2
+Text GLabel 2580 6590 2    47   UnSpc ~ 0
+LIGHT_INT
+Wire Wire Line
+	2405 6590 2580 6590
 $EndSCHEMATC
