File: pcbs/proj/led_driver.kicad_pcb (KiCad board)
At the start: 4 copper layers, 100 x 82.5 mm, 348 parts, among them J1 Conn_02x32_Counter_Clockwise, J2 Conn_02x03_Odd_Even, J3 Conn_01x05, J4 Conn_02x05_Odd_Even, J5 Barrel_Jack, J6 Conn_02x19_Odd_Even, J7 Conn_02x19_Odd_Even, J8 Conn_01x07, Q1 MBT3904DW1, Q10 MBT3904DW1, Q11 MBT3904DW1, Q12 MBT3904DW1, Q13 MBT3904DW1, Q14 MBT3904DW1, Q15 MBT3904DW1, Q16 MBT3904DW1, Q17 MBT3904DW1, Q18 MBT3904DW1, Q19 MBT3904DW1, Q2 MBT3904DW1, Q20 MBT3904DW1, Q21 MBT3904DW1, Q22 MBT3904DW1, Q23 MBT3904DW1, Q24 MBT3904DW1, Q25 MBT3904DW1, Q26 MBT3904DW1, Q27 MBT3904DW1, Q28 MBT3904DW1, Q29 MBT3904DW1, Q3 MBT3904DW1, Q30 MBT3904DW1, Q31 MBT3904DW1, Q32 MBT3904DW1, Q4 MBT3904DW1, Q5 MBT3904DW1, Q6 MBT3904DW1, Q7 MBT3904DW1, Q8 MBT3904DW1, Q9 MBT3904DW1, SW1 MY_SW_Push_Dual, SW2 Rotary_Encoder, SW3 Rotary_Encoder, U1 LM324QT, U10 LM324QT, U11 LM324QT, U12 LM324QT, U13 LM324QT, U14 LM324QT, U15 LM324QT, U16 LM324QT, U17 LM324QT, U18 LM324QT, U19 LM324QT, U2 LM324QT, U20 LM324QT, U21 LM324QT, U22 LM324QT, U23 LM324QT, U24 LM324QT, U25 LM324QT, U26 LM324QT, U27 LM324QT, U28 LM324QT, U29 LM324QT, U3 LM324QT, U30 LM324QT, U31 LM324QT, U32 LM324QT, U33 DAC101C085, U34 TS30011/12/13, U4 LM324QT, U5 LM324QT, U6 LM324QT, U7 LM324QT, U8 LM324QT, U9 LM324QT

Commit message: Some progress layouting the beast today.
Parts:
- R198: footprint Resistors_SMD:R_1206 -> Resistors_SMD:R_2512_HandSoldering
- moved TP6 164.6 mm to (174.5, 102.5)
- moved TP8 163.1 mm to (174.5, 97.7)
- moved TP5 159.6 mm to (168.3, 105.0)
- moved TP1 142.2 mm to (150.1, 103.8)
- moved TP2 136.1 mm to (138.8, 113.4)
- moved TP4 134.4 mm to (140.0, 107.4)
- moved D4 127.5 mm to (133.6, 107.4), turned to 0 degrees
- moved R199 126.4 mm to (136.5, 114.2)
- moved D1 125.8 mm to (135.8, 112.4)
- moved R3 123.7 mm to (158.9, 104.9), turned to 270 degrees
- moved J3 123.7 mm to (128.9, 92.8)
- moved R201 123.7 mm to (130.4, 107.4)
- moved R4 122.7 mm to (167.1, 103.0)
- moved Q13 122.5 mm to (148.0, 56.4)
- moved Q25 122.5 mm to (192.2, 56.4)
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Routing:
- net VSIG: track 0.00 -> 281.9 mm, vias 0 -> 64
- net +3V3: track 0.00 -> 119.8 mm
- net PC9: track 0.00 -> 91.6 mm, vias 0 -> 1
- net LED_N_54: track 0.00 -> 86.9 mm, vias 0 -> 1
- net LED_N_53: track 0.00 -> 78.4 mm, vias 0 -> 1
- net LED_N_56: track 0.00 -> 77.5 mm, vias 0 -> 1
- net PC10: track 0.00 -> 75.2 mm
- net LED_N_58: track 0.00 -> 74.5 mm, vias 0 -> 1
- net LED_N_55: track 0.00 -> 73.3 mm, vias 0 -> 1
- net LED_N_60: track 0.00 -> 70.3 mm, vias 0 -> 1
- net LED_N_57: track 0.00 -> 68.2 mm, vias 0 -> 1
- net LED_N_64: track 0.00 -> 63.5 mm, vias 0 -> 1
- net LED_N_62: track 0.00 -> 63.2 mm, vias 0 -> 1
- net LED_N_59: track 0.00 -> 63.1 mm, vias 0 -> 1
- net LED_N_07: track 0.00 -> 61.2 mm
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- added copper zone on F.Cu, net GND
- added copper zone on S2.Cu, net GND
- removed copper zone on GND.Cu, net GND
Other:
- net class Default: clearance 0.15 -> 0.19
- rule trace_clearance: 0.15 -> 0.19

Commit message: Started eliminating DRC errors.
Parts:
- added REF**: Stitching-Via-0.4-0.7, MyVias:Stitchging-Via-0.4-0.7, F.Cu at (157.8, 109.5)
- added REF**: Stitching-Via-0.4-0.7, MyVias:Stitchging-Via-0.4-0.7, F.Cu at (132.3, 106.9)
- added REF**: Stitching-Via-0.4-0.7, MyVias:Stitchging-Via-0.4-0.7, F.Cu at (133.6, 106.9)
- added REF**: Stitching-Via-0.4-0.7, MyVias:Stitchging-Via-0.4-0.7, F.Cu at (148.0, 95.1)
- added REF**: Stitching-Via-0.4-0.7, MyVias:Stitchging-Via-0.4-0.7, F.Cu at (146.7, 95.1)
- added REF**: Stitching-Via-0.4-0.7, MyVias:Stitchging-Via-0.4-0.7, F.Cu at (145.4, 95.1)
- added REF**: Stitching-Via-0.4-0.7, MyVias:Stitchging-Via-0.4-0.7, F.Cu at (142.9, 95.1)
- added REF**: Stitching-Via-0.4-0.7, MyVias:Stitchging-Via-0.4-0.7, F.Cu at (144.1, 95.1)
- added REF**: Stitching-Via-0.4-0.7, MyVias:Stitchging-Via-0.4-0.7, F.Cu at (136.5, 95.1)
- added REF**: Stitching-Via-0.4-0.7, MyVias:Stitchging-Via-0.4-0.7, F.Cu at (135.3, 95.1)
- added REF**: Stitching-Via-0.4-0.7, MyVias:Stitchging-Via-0.4-0.7, F.Cu at (134.0, 95.1)
- added REF**: Stitching-Via-0.4-0.7, MyVias:Stitchging-Via-0.4-0.7, F.Cu at (156.5, 109.5)
- added REF**: Stitching-Via-0.4-0.7, MyVias:Stitchging-Via-0.4-0.7, F.Cu at (137.8, 95.1)
- added REF**: Stitching-Via-0.4-0.7, MyVias:Stitchging-Via-0.4-0.7, F.Cu at (149.4, 106.7)
- added REF**: Stitching-Via-0.4-0.7, MyVias:Stitchging-Via-0.4-0.7, F.Cu at (149.4, 105.4)
- added REF**: Stitching-Via-0.4-0.7, MyVias:Stitchging-Via-0.4-0.7, F.Cu at (149.4, 104.1)
- added REF**: Stitching-Via-0.4-0.7, MyVias:Stitchging-Via-0.4-0.7, F.Cu at (149.4, 95.2)
- added REF**: Stitching-Via-0.4-0.7, MyVias:Stitchging-Via-0.4-0.7, F.Cu at (149.4, 96.5)
- added REF**: Stitching-Via-0.4-0.7, MyVias:Stitchging-Via-0.4-0.7, F.Cu at (149.4, 97.8)
- added REF**: Stitching-Via-0.4-0.7, MyVias:Stitchging-Via-0.4-0.7, F.Cu at (149.4, 99.1)
- added REF**: Stitching-Via-0.4-0.7, MyVias:Stitchging-Via-0.4-0.7, F.Cu at (129.8, 102.6)
- added REF**: Stitching-Via-0.4-0.7, MyVias:Stitchging-Via-0.4-0.7, F.Cu at (129.8, 101.3)
- added REF**: Stitching-Via-0.4-0.7, MyVias:Stitchging-Via-0.4-0.7, F.Cu at (155.3, 109.5)
- added REF**: Stitching-Via-0.4-0.7, MyVias:Stitchging-Via-0.4-0.7, F.Cu at (129.8, 100.1)
- added REF**: Stitching-Via-0.4-0.7, MyVias:Stitchging-Via-0.4-0.7, F.Cu at (129.8, 96.3)
- added REF**: Stitching-Via-0.4-0.7, MyVias:Stitchging-Via-0.4-0.7, F.Cu at (129.8, 97.5)
- added REF**: Stitching-Via-0.4-0.7, MyVias:Stitchging-Via-0.4-0.7, F.Cu at (129.8, 98.8)
- added REF**: Stitching-Via-0.4-0.7, MyVias:Stitchging-Via-0.4-0.7, F.Cu at (129.8, 106.4)
- added REF**: Stitching-Via-0.4-0.7, MyVias:Stitchging-Via-0.4-0.7, F.Cu at (129.8, 105.2)
- added REF**: Stitching-Via-0.4-0.7, MyVias:Stitchging-Via-0.4-0.7, F.Cu at (129.8, 103.9)
- added REF**: Stitching-Via-0.4-0.7, MyVias:Stitchging-Via-0.4-0.7, F.Cu at (151.4, 109.5)
- added REF**: Stitching-Via-0.4-0.7, MyVias:Stitchging-Via-0.4-0.7, F.Cu at (152.7, 109.5)
- added REF**: Stitching-Via-0.4-0.7, MyVias:Stitchging-Via-0.4-0.7, F.Cu at (154.0, 109.5)
- added REF**: Stitching-Via-0.4-0.7, MyVias:Stitchging-Via-0.4-0.7, F.Cu at (136.1, 106.9)
- added REF**: Stitching-Via-0.4-0.7, MyVias:Stitchging-Via-0.4-0.7, F.Cu at (134.9, 106.9)
- added REF**: Stitching-Via-0.4-0.7, MyVias:Stitchging-Via-0.4-0.7, F.Cu at (131.1, 106.9)
- R198: footprint Resistors_SMD:R_2512_HandSoldering -> Resistors_SMD:R_1206
- moved J8 21.1 mm to (151.1, 90.0), turned to 90 degrees
- moved C136 11.4 mm to (136.1, 96.6), turned to 90 degrees
- moved TP5 11.1 mm to (174.5, 95.8)
- moved TP6 11.0 mm to (174.5, 91.4)
- moved TP2 9.90 mm to (129.0, 111.9)
- moved R199 6.79 mm to (129.8, 115.1)
- moved D1 6.05 mm to (129.8, 113.4)
- moved R200 5.88 mm to (122.3, 98.0), turned to 180 degrees
- moved R201 3.70 mm to (131.4, 103.9), turned to 90 degrees
- moved D4 3.59 mm to (133.1, 103.9), turned to 90 degrees
- moved J2 3.45 mm to (163.8, 94.6)
- moved D3 3.44 mm to (122.3, 96.5)
- moved C1 3.37 mm to (164.2, 107.7)
- moved C3 3.37 mm to (167.5, 107.7)
- moved C2 3.37 mm to (165.9, 107.7)
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Connections:
- J2 pad 5: GND -> (no net)
- J3 pad 5: (no net) -> LIGHT_INT
- J6 pad 3: (no net) -> LIGHT_INT
- U1 pad 17: (no net) -> GND
- U10 pad 17: (no net) -> GND
- U11 pad 17: (no net) -> GND
- U12 pad 17: (no net) -> GND
- U13 pad 17: (no net) -> GND
- U14 pad 17: (no net) -> GND
- U15 pad 17: (no net) -> GND
- U16 pad 17: (no net) -> GND
- U17 pad 17: (no net) -> GND
- U18 pad 17: (no net) -> GND
- U19 pad 17: (no net) -> GND
- U2 pad 17: (no net) -> GND
- U20 pad 17: (no net) -> GND
- U21 pad 17: (no net) -> GND
- U22 pad 17: (no net) -> GND
- U23 pad 17: (no net) -> GND
- U24 pad 17: (no net) -> GND
- U25 pad 17: (no net) -> GND
- U26 pad 17: (no net) -> GND
- U27 pad 17: (no net) -> GND
- U28 pad 17: (no net) -> GND
- U29 pad 17: (no net) -> GND
- U3 pad 17: (no net) -> GND
- U30 pad 17: (no net) -> GND
- U31 pad 17: (no net) -> GND
- U32 pad 17: (no net) -> GND
- U33 pad 3: I2C_SDA -> I2C_SCL
- U33 pad 4: I2C_SCL -> I2C_SDA
- U34 pad 17: (no net) -> GND
- U4 pad 17: (no net) -> GND
- U5 pad 17: (no net) -> GND
- U6 pad 17: (no net) -> GND
- U7 pad 17: (no net) -> GND
- U8 pad 17: (no net) -> GND
- U9 pad 17: (no net) -> GND
Routing:
- net PC11: track 1.52 -> 109.1 mm, vias 0 -> 1
- net +3V3: track 119.8 -> 211.1 mm, vias 0 -> 2
- net PC12: track 1.52 -> 89.9 mm
- net I2C_SDA: track 8.30 -> 72.9 mm, vias 0 -> 1
- net VSIG: track 281.9 -> 330.7 mm
- net CS_OLED: track 0.00 -> 46.9 mm
- net GND: track 56.2 -> 99.5 mm, vias 55 -> 90
- net E5V: track 30.4 -> 63.1 mm
- net I2C_SCL: track 37.7 -> 69.5 mm, vias 1 -> 2
- net PA8: track 0.00 -> 30.4 mm
- net DC_OLED: track 0.00 -> 28.1 mm
- net LIGHT_INT: track 0.00 -> 26.5 mm
- net PA7: track 0.00 -> 24.9 mm
- net PA5: track 0.30 -> 24.5 mm
- net V18: track 49.8 -> 61.0 mm, vias 31 -> 37
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