File: pcbs/adapter_board/adapter_board.kicad_pcb (KiCad board)
At the start: 2 copper layers, 100 x 45 mm, 71 parts, among them J1 Conn_02x32_Counter_Clockwise, J2 Conn_02x05_Odd_Even

Commit message: Produced Gerber files for both boards. Ready for production.
Other:
- board text added: "Power Supply"
- board text removed: "18V"
Changed lines of the file:
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@@
     (links 73)
     (no_connects 0)
-    (area 82.733287 69.924999 206.953715 123.905001)
+    (area 95.924999 69.924999 196.075001 115.075001)
     (thickness 1.6)
     (drawings 21)
@@
     (pad_drill 0.762)
     (pad_to_mask_clearance 0.2)
-    (aux_axis_origin 0 0)
+    (aux_axis_origin 96 70)
+    (grid_origin 96 70)
     (visible_elements FFFFFF7F)
     (pcbplotparams
@@
       (viasonmask false)
       (mode 1)
-      (useauxorigin false)
+      (useauxorigin true)
       (hpglpennumber 1)
       (hpglpenspeed 20)
@@
     (effects (font (size 1.5 1.5) (thickness 0.3)) (justify mirror))
   )
-  (gr_text 18V (at 104.394 99.822) (layer F.SilkS)
+  (gr_text "Power \nSupply" (at 104.509 98.829) (layer F.SilkS)
     (effects (font (size 1.5 1.5) (thickness 0.3)))
   )
