File: pcbs/extension_board/LEDDriver.sch (KiCad schematic (older format))
At the start: 12 parts, among them J1 Conn_02x32_Counter_Clockwise, J2 Conn_02x03_Odd_Even, J3 Conn_01x05, U33 DAC101C085

Commit message: Added more OS files to be tracked. Port them now to the STM32.
Parts:
- J2: Digikey TSW-103-07-G-D -> (none); Samtec (none) -> TSW-103-07-G-D
Changed lines of the file:
@@
 VDAC
 $Comp
-L GND #PWR3
+L GND #PWR01
 U 1 1 5A10F0A9
 P 9100 2845
-F 0 "#PWR3" H 9100 2595 50  0001 C CNN
+F 0 "#PWR01" H 9100 2595 50  0001 C CNN
 F 1 "GND" H 9100 2695 50  0000 C CNN
 F 2 "" H 9100 2845 50  0000 C CNN
@@
 $EndComp
 $Comp
-L GND #PWR1
+L GND #PWR02
 U 1 1 5A142088
 P 7570 4080
-F 0 "#PWR1" H 7570 3830 50  0001 C CNN
+F 0 "#PWR02" H 7570 3830 50  0001 C CNN
 F 1 "GND" H 7570 3930 50  0000 C CNN
 F 2 "" H 7570 4080 50  0000 C CNN
@@
 F 2 "Pin_Headers:Pin_Header_Straight_2x03_Pitch2.54mm" H 8210 3830 50  0001 C CNN
 F 3 "" H 8210 3830 50  0001 C CNN
-F 4 "TSW-103-07-G-D" H 8210 3830 60  0001 C CNN "Digikey"
+F 4 "TSW-103-07-G-D" H 8210 3830 60  0001 C CNN "Samtec"
 	1    8210 3830
 	1    0    0    -1
@@
 $EndComp
 $Comp
-L GND #PWR2
+L GND #PWR03
 U 1 1 5A15B686
 P 8840 4080
-F 0 "#PWR2" H 8840 3830 50  0001 C CNN
+F 0 "#PWR03" H 8840 3830 50  0001 C CNN
 F 1 "GND" H 8840 3930 50  0000 C CNN
 F 2 "" H 8840 4080 50  0000 C CNN
