File: pcbs/extension_board/power.sch (KiCad schematic (older format))
At the start: 23 parts, among them J4 Conn_02x05_Odd_Even, J5 Barrel_Jack, U34 TS30011/12/13

Commit message: Produced Gerber files for both boards. Ready for production.
Other:
- note added: "4.5 V to 24 V, max. 1A, 1 MHz"
Changed lines of the file:
@@
 Text Notes 4060 1605 0    60   ~ 0
 Current Rating (IPC 2221)\n----------------------\nMax. Expected Current = 64 * 0.05 A = 3.2 A \nAbs. Max. Current (dT = 10 K, W = 1.6 mm) = 3.36 A
+Text Notes 1700 6650 0    60   ~ 0
+4.5 V to 24 V, max. 1A, 1 MHz
 $EndSCHEMATC

Commit message: Added more OS files to be tracked. Port them now to the STM32.
Parts:
- R200: Digikey 1276-6153-1-ND -> 311-20GRCT-ND
- R201: Digikey 311-360GRCT-ND -> 311-20GRCT-ND
Changed lines of the file:
@@
 $EndComp
 $Comp
-L GND #PWR294
+L GND #PWR0292
 U 1 1 5A0AD8CE
 P 5090 3180
-F 0 "#PWR294" H 5090 2930 50  0001 C CNN
+F 0 "#PWR0292" H 5090 2930 50  0001 C CNN
 F 1 "GND" H 5090 3030 50  0000 C CNN
 F 2 "" H 5090 3180 50  0001 C CNN
@@
 V18
 $Comp
-L GND #PWR295
+L GND #PWR0293
 U 1 1 5A0B8173
 P 5115 5940
-F 0 "#PWR295" H 5115 5690 50  0001 C CNN
+F 0 "#PWR0293" H 5115 5690 50  0001 C CNN
 F 1 "GND" H 5115 5790 50  0000 C CNN
 F 2 "" H 5115 5940 50  0001 C CNN
@@
 FB
 $Comp
-L GND #PWR293
+L GND #PWR0294
 U 1 1 5A0B8CE5
 P 4690 5160
-F 0 "#PWR293" H 4690 4910 50  0001 C CNN
+F 0 "#PWR0294" H 4690 4910 50  0001 C CNN
 F 1 "GND" H 4690 5010 50  0000 C CNN
 F 2 "" H 4690 5160 50  0001 C CNN
@@
 $EndComp
 $Comp
-L GND #PWR292
+L GND #PWR0295
 U 1 1 5A0BC4D5
 P 1985 5940
-F 0 "#PWR292" H 1985 5690 50  0001 C CNN
+F 0 "#PWR0295" H 1985 5690 50  0001 C CNN
 F 1 "GND" H 1985 5790 50  0000 C CNN
 F 2 "" H 1985 5940 50  0001 C CNN
@@
 F 2 "Resistors_SMD:R_0603" V 8700 4560 50  0001 C CNN
 F 3 "" H 8770 4560 50  0001 C CNN
-F 4 "311-360GRCT-ND" V 8770 4560 60  0001 C CNN "Digikey"
+F 4 "311-20GRCT-ND " V 8770 4560 60  0001 C CNN "Digikey"
 	1    8770 4560
 	-1   0    0    -1
 $EndComp
 $Comp
-L GND #PWR297
+L GND #PWR0296
 U 1 1 5A0C1EE8
 P 8770 4770
-F 0 "#PWR297" H 8770 4520 50  0001 C CNN
+F 0 "#PWR0296" H 8770 4520 50  0001 C CNN
 F 1 "GND" H 8770 4620 50  0000 C CNN
 F 2 "" H 8770 4770 50  0001 C CNN
@@
 F 2 "Resistors_SMD:R_0603" V 8670 2690 50  0001 C CNN
 F 3 "" H 8740 2690 50  0001 C CNN
-F 4 "1276-6153-1-ND" V 8740 2690 60  0001 C CNN "Digikey"
+F 4 "311-20GRCT-ND " V 8740 2690 60  0001 C CNN "Digikey"
 	1    8740 2690
 	-1   0    0    -1
 $EndComp
 $Comp
-L GND #PWR296
+L GND #PWR0297
 U 1 1 5A0EF3E8
 P 8740 2900
-F 0 "#PWR296" H 8740 2650 50  0001 C CNN
+F 0 "#PWR0297" H 8740 2650 50  0001 C CNN
 F 1 "GND" H 8740 2750 50  0000 C CNN
 F 2 "" H 8740 2900 50  0001 C CNN
@@
 3V3
 $Comp
-L PWR_FLAG #FLG1
+L PWR_FLAG #FLG0298
 U 1 1 5A107991
 P 5025 3960
-F 0 "#FLG1" H 5025 4035 50  0001 C CNN
+F 0 "#FLG0298" H 5025 4035 50  0001 C CNN
 F 1 "PWR_FLAG" H 5025 4110 50  0000 C CNN
 F 2 "" H 5025 3960 50  0001 C CNN
@@
 V18
 $Comp
-L PWR_FLAG #FLG2
+L PWR_FLAG #FLG0299
 U 1 1 5A107A22
 P 5475 3960
-F 0 "#FLG2" H 5475 4035 50  0001 C CNN
+F 0 "#FLG0299" H 5475 4035 50  0001 C CNN
 F 1 "PWR_FLAG" H 5475 4110 50  0000 C CNN
 F 2 "" H 5475 3960 50  0001 C CNN
